File: VR-Shield.kicad_sch (KiCad schematic)
At the start: 19 parts, among them Q1 IRF7404, Q2 BC847, U1 ESP32 WROOM32 Devkit, U2 MCP73831-2-OT

Commit message: Fixed issues with pad size and distance Please enter the commit message for your changes. Lines starting
Parts:
- removed CB1: RST, Button_Switch_THT:SW_Tactile_Straight_KSA0Axx1LFTR, symbol Device:CircuitBreaker_1P
- P1, P2, P3, P4: footprint Connector_TE-Connectivity:TE_Micro-MaTch_215079-4_2x02_P1.27mm_Vertical -> Custom:TE_Micro-MaTch_215079-4_2x02_P1.27mm_Vertical
Connections:
- net GND: no longer U1.14 (GND)
- no-connect marks 30 -> 31
Changed lines of the file:
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@@
   (junction (at 214.63 100.33) (diameter 0) (color 0 0 0 0)
   )
-  (junction (at 95.25 115.57) (diameter 0) (color 0 0 0 0)
-  )
   (junction (at 232.41 100.33) (diameter 0) (color 0 0 0 0)
   )
@@
   (junction (at 197.485 113.03) (diameter 0) (color 0 0 0 0)
   )
+  (no_connect (at 111.76 115.57))
   (no_connect (at 111.76 120.65))
   (no_connect (at 180.34 105.41))
@@
     (stroke (width 0) (type default))
   )
-  (wire (pts (xy 94.615 115.57) (xy 95.25 115.57))
-    (stroke (width 0) (type default))
-  )
   (wire (pts (xy 48.895 50.165) (xy 48.895 32.385))
     (stroke (width 0) (type default))
@@
     (stroke (width 0) (type default))
   )
-  (wire (pts (xy 95.25 115.57) (xy 111.76 115.57))
-    (stroke (width 0) (type default))
-  )
   (wire (pts (xy 209.55 87.63) (xy 227.33 87.63))
     (stroke (width 0) (type default))
   )
-  (wire (pts (xy 95.25 85.09) (xy 111.76 85.09))
-    (stroke (width 0) (type default))
-  )
   (wire (pts (xy 105.41 97.79) (xy 111.76 97.79))
     (stroke (width 0) (type default))
@@
     (stroke (width 0) (type default))
   )
-  (wire (pts (xy 95.25 87.63) (xy 95.25 85.09))
-    (stroke (width 0) (type default))
-  )
   (wire (pts (xy 250.19 100.33) (xy 232.41 100.33))
     (stroke (width 0) (type default))
@@
     (stroke (width 0) (type default))
   )
-  (wire (pts (xy 95.25 102.87) (xy 95.25 115.57))
-    (stroke (width 0) (type default))
-  )
   (wire (pts (xy 189.23 100.33) (xy 180.34 100.33))
     (stroke (width 0) (type default))
   )
   (wire (pts (xy 194.31 95.25) (xy 194.31 73.025))
-    (stroke (width 0) (type default))
-  )
-  (wire (pts (xy 95.25 140.97) (xy 95.25 115.57))
     (stroke (width 0) (type default))
   )
@@
       (effects (font (size 1.27 1.27)))
     )
-    (property "Footprint" "Connector_TE-Connectivity:TE_Micro-MaTch_215079-4_2x02_P1.27mm_Vertical" (at 193.04 73.025 0)
+    (property "Footprint" "Custom:TE_Micro-MaTch_215079-4_2x02_P1.27mm_Vertical" (at 193.04 73.025 0)
       (effects (font (size 1.27 1.27)) hide)
     )
@@
       (effects (font (size 1.27 1.27)))
     )
-    (property "Footprint" "Connector_TE-Connectivity:TE_Micro-MaTch_215079-4_2x02_P1.27mm_Vertical" (at 228.6 73.025 0)
+    (property "Footprint" "Custom:TE_Micro-MaTch_215079-4_2x02_P1.27mm_Vertical" (at 228.6 73.025 0)
       (effects (font (size 1.27 1.27)) hide)
     )
@@
     )
   )
-  (symbol (lib_id "Device:CircuitBreaker_1P") (at 95.25 95.25 0) (unit 1)
-    (in_bom yes) (on_board yes) (dnp no)
-    (property "Reference" "CB1" (at 96.52 94.615 0)
-      (effects (font (size 1.27 1.27)) (justify left))
-    )
-    (property "Value" "RST" (at 96.52 97.155 0)
-      (effects (font (size 1.27 1.27)) (justify left))
-    )
-    (property "Footprint" "Button_Switch_THT:SW_Tactile_Straight_KSA0Axx1LFTR" (at 95.25 95.25 0)
-      (effects (font (size 1.27 1.27)) hide)
-    )
-    (property "Datasheet" "~" (at 95.25 95.25 0)
-      (effects (font (size 1.27 1.27)) hide)
-    )
-    (pin "1")
-    (pin "2")
-    (instances
-      (project "VR-Shield"
-        (path "/b4b07443-399e-4a24-8592-985a350f897a"
-          (reference "CB1") (unit 1)
-        )
-      )
-    )
-  )
   (symbol (lib_id "I2CSockets:I2CSocket") (at 210.82 73.025 180) (unit 1)
     (in_bom yes) (on_board yes) (dnp no) (fields_autoplaced)
@@
       (effects (font (size 1.27 1.27)))
     )
-    (property "Footprint" "Connector_TE-Connectivity:TE_Micro-MaTch_215079-4_2x02_P1.27mm_Vertical" (at 210.82 73.025 0)
+    (property "Footprint" "Custom:TE_Micro-MaTch_215079-4_2x02_P1.27mm_Vertical" (at 210.82 73.025 0)
       (effects (font (size 1.27 1.27)) hide)
     )
@@
         (path "/b4b07443-399e-4a24-8592-985a350f897a"
           (reference "R5") (unit 1)
-        )
-      )
-    )
-  )
-  (symbol (lib_id "power:GND") (at 95.25 140.97 0) (unit 1)
-    (in_bom yes) (on_board yes) (dnp no) (fields_autoplaced)
-    (property "Reference" "#PWR01" (at 95.25 147.32 0)
-      (effects (font (size 1.27 1.27)) hide)
-    )
-    (property "Value" "GND" (at 95.25 145.415 0)
-      (effects (font (size 1.27 1.27)))
-    )
-    (property "Footprint" "" (at 95.25 140.97 0)
-      (effects (font (size 1.27 1.27)) hide)
-    )
-    (property "Datasheet" "" (at 95.25 140.97 0)
-      (effects (font (size 1.27 1.27)) hide)
-    )
-    (pin "1")
-    (instances
-      (project "VR-Shield"
-        (path "/b4b07443-399e-4a24-8592-985a350f897a"
-          (reference "#PWR01") (unit 1)
         )
       )
@@
       (effects (font (size 1.27 1.27)))
     )
-    (property "Footprint" "Connector_TE-Connectivity:TE_Micro-MaTch_215079-4_2x02_P1.27mm_Vertical" (at 246.38 73.025 0)
-      (effects (font (size 1.27 1.27)) hide)
-    )
+    (property "Footprint" "Custom:TE_Micro-MaTch_215079-4_2x02_P1.27mm_Vertical" (at 246.38 73.025 0)
+      (effects (font (size 1.27 1.27)) hide)
+    )

Commit message: t V03!!!!
Parts:
- removed BT1: Battery_Cell, Connector_JST:JST_SH_BM02B-SRSS-TB_1x02-1MP_P1.00mm_Vertical, symbol Device:Battery_Cell
- removed C1: C, Capacitor_SMD:C_0805_2012Metric_Pad1.18x1.45mm_HandSolder, symbol Device:C
- removed C2: 4,7u, Capacitor_SMD:C_0805_2012Metric_Pad1.18x1.45mm_HandSolder, symbol Device:C
- removed D2: GREEN, LED_SMD:LED_0805_2012Metric_Pad1.15x1.40mm_HandSolder, symbol Device:LED
- removed P1, P2, P3, P4: ~, Custom:TE_Micro-MaTch_215079-4_2x02_P1.27mm_Vertical, symbol I2CSockets:I2CSocket
- removed R4: 10k, Resistor_SMD:R_0805_2012Metric_Pad1.20x1.40mm_HandSolder, symbol Device:R
- removed R5: 470, Resistor_SMD:R_0805_2012Metric_Pad1.20x1.40mm_HandSolder, symbol Device:R
- removed U2: MCP73831-2-OT, Package_TO_SOT_SMD:SOT-23-5, symbol Battery_Management:MCP73831-2-OT
- added J1, J5: Double I2C Socket, Custom:Custom Socket I2C, symbol Connector:Conn_01x12_Socket
Connections:
- net GND: now also J1.1 (Pin_1), J1.7 (Pin_7), J5.1 (Pin_1), J5.7 (Pin_7)
- net SCL: now reaches U1.36 (GPIO22)
- net SCL: now also J1.2 (Pin_2), J1.8 (Pin_8), J5.2 (Pin_2), J5.8 (Pin_8)
- net SDA: now reaches U1.33 (GPIO21)
- net SDA: now also J1.11 (Pin_11), J1.5 (Pin_5), J5.11 (Pin_11), J5.5 (Pin_5)
- net VCC: now reaches Q1.5 (D), Q1.6 (D), Q1.7 (D), Q1.8 (D)
- net VCC: now also J1.12 (Pin_12), J1.6 (Pin_6), J5.12 (Pin_12), J5.6 (Pin_6)
- no-connect marks 31 -> 41

Commit message: User friendlyness improved
Connections:
- net at U1.31 (GPIO19): no longer R2.1
- net 5V renamed +5V
- new net CTRL: R2.1
- no-connect marks 41 -> 40
Other:
- note added: "I2C Connector"
- note added: "I2C Power Supply"
- note added: "MCU"
- moved on the sheet: D1, J1, J5, Q1, Q2, R1, R2, R3, U1
